File: psu/psu.brd (EAGLE design)
At the start: 99.1 x 78.7 mm, 39 parts, among them IC1 7815T, IC2 7915T, IC3 7812T, IC4 7912T, IC5 7805T, J1 15VAC, J2 POWER_SW

Commit message: Loading resistors for the PSU
Parts:
- added R1, R2, R3, R4, R5: 2.4k, SparkFun-Resistors:0805
Connections:
- net +12V: now also R2.1
- net +15V: now also R1.1
- net +5V: now also R3.1
- net -12V: now also R4.1
- net -15V: now also R5.1
- net GND: now also R1.2, R2.2, R3.2, R4.2, R5.2
Routing:
- net +15V: track 51.3 -> 53.6 mm
- net -12V: track 94.8 -> 97.1 mm
- net +5V: track 44.8 -> 47.0 mm
- net -15V: track 59.5 -> 61.6 mm
- net GND: track 15.9 -> 14.1 mm
- net +12V: track 82.3 -> 84.0 mm
Changed lines of the file:
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@@
 <element name="JP1" library="pinhead" package="2X07" value="" x="83.82" y="39.37" rot="R270"/>
 <element name="D11" library="diode" package="DO41-10" value="1N4004" x="73.66" y="66.04" rot="R270"/>
+<element name="R1" library="SparkFun-Resistors" package="0805" value="2.4k" x="47.879" y="46.609" rot="MR90"/>
+<element name="R2" library="SparkFun-Resistors" package="0805" value="2.4k" x="20.32" y="43.18" rot="MR270"/>
+<element name="R3" library="SparkFun-Resistors" package="0805" value="2.4k" x="81.28" y="53.34" rot="MR270"/>
+<element name="R4" library="SparkFun-Resistors" package="0805" value="2.4k" x="19.685" y="19.05" rot="MR270"/>
+<element name="R5" library="SparkFun-Resistors" package="0805" value="2.4k" x="50.165" y="19.177" rot="MR270"/>
 </elements>
 <signals>
@@
 <vertex x="110.49" y="83.82"/>
 </polygon>
-<via x="3.81" y="19.685" extent="1-16" drill="1.524"/>
-<via x="19.685" y="19.685" extent="1-16" drill="1.524"/>
-<wire x1="19.685" y1="19.685" x2="3.81" y2="19.685" width="1.016" layer="1"/>
+<via x="32.385" y="3.048" extent="1-16" drill="1.524"/>
+<via x="32.385" y="17.145" extent="1-16" drill="1.524"/>
+<wire x1="32.385" y1="17.145" x2="32.385" y2="3.048" width="1.016" layer="1"/>
+<contactref element="R1" pad="2"/>
+<contactref element="R2" pad="2"/>
+<contactref element="R3" pad="2"/>
+<contactref element="R4" pad="2"/>
+<contactref element="R5" pad="2"/>
 </signal>
 <signal name="+AC">
@@
 <wire x1="69.215" y1="46.99" x2="82.55" y2="46.99" width="1.4224" layer="16"/>
 <wire x1="53.975" y1="45.72" x2="56.515" y2="45.72" width="1.4224" layer="16"/>
+<contactref element="R1" pad="1"/>
+<wire x1="50.165" y1="45.72" x2="47.89" y2="45.72" width="1.27" layer="16"/>
+<wire x1="47.89" y1="45.72" x2="47.879" y2="45.709" width="1.27" layer="16"/>
 </signal>
 <signal name="-15V">
@@
 <wire x1="62.865" y1="24.765" x2="69.85" y2="31.75" width="1.4224" layer="16"/>
 <wire x1="69.85" y1="31.75" x2="82.55" y2="31.75" width="1.4224" layer="16"/>
+<contactref element="R5" pad="1"/>
+<wire x1="50.165" y1="22.225" x2="50.165" y2="20.077" width="1.27" layer="16"/>
 </signal>
 <signal name="+12V">
@@
 <wire x1="46.99" y1="41.275" x2="42.545" y2="45.72" width="1.4224" layer="16"/>
 <wire x1="42.545" y1="45.72" x2="26.035" y2="45.72" width="1.4224" layer="16"/>
+<contactref element="R2" pad="1"/>
+<wire x1="20.32" y1="45.72" x2="20.32" y2="44.08" width="1.27" layer="16"/>
 </signal>
 <signal name="-12V">
@@
 <wire x1="33.02" y1="26.035" x2="31.75" y2="24.765" width="1.4224" layer="16"/>
 <wire x1="31.75" y1="24.765" x2="26.67" y2="24.765" width="1.4224" layer="16"/>
+<contactref element="R4" pad="1"/>
+<wire x1="19.685" y1="22.225" x2="19.685" y2="19.95" width="1.27" layer="16"/>
 </signal>
 <signal name="+5V">
@@
 <wire x1="85.725" y1="56.515" x2="90.17" y2="52.07" width="0.6096" layer="1"/>
 <wire x1="90.17" y1="52.07" x2="90.17" y2="41.91" width="0.6096" layer="1"/>
+<contactref element="R3" pad="1"/>
+<wire x1="81.28" y1="56.515" x2="81.28" y2="54.24" width="1.27" layer="16"/>
 <wire x1="77.47" y1="60.96" x2="77.47" y2="63.5" width="0" layer="19" extent="1-1"/>
 </signal>

Commit message: psu rev 2: fix disconnected nets, add led
Parts:
- added LED1: (no value), led:LED3MM
Connections:
- net +5V: now also LED1.A
- net GND: now also LED1.K
Routing:
- net +5V: track 47.0 -> 55.2 mm
- net +AC: track 117.4 -> 119.9 mm
Changed lines of the file:
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@@
 <?xml version="1.0" encoding="utf-8"?>
 <!DOCTYPE eagle SYSTEM "eagle.dtd">
-<eagle version="7.5.0">
+<eagle version="7.6.0">
 <drawing>
 <settings>
@@
 <element name="R4" library="SparkFun-Resistors" package="0805" value="2.4k" x="19.685" y="19.05" rot="MR270"/>
 <element name="R5" library="SparkFun-Resistors" package="0805" value="2.4k" x="50.165" y="19.177" rot="MR270"/>
+<element name="LED1" library="led" package="LED3MM" value="" x="77.47" y="39.37" rot="R270"/>
 </elements>
 <signals>
@@
 <contactref element="R4" pad="2"/>
 <contactref element="R5" pad="2"/>
+<contactref element="LED1" pad="K"/>
 </signal>
 <signal name="+AC">
@@
 <wire x1="53.34" y1="66.04" x2="52.705" y2="65.405" width="1.6764" layer="16"/>
 <wire x1="52.705" y1="65.405" x2="52.705" y2="55.88" width="1.6764" layer="16"/>
-<wire x1="77.47" y1="71.12" x2="77.47" y2="68.58" width="0" layer="19" extent="1-1"/>
+<wire x1="77.47" y1="71.12" x2="77.47" y2="68.58" width="1.4224" layer="16"/>
 </signal>
 <signal name="-AC">
@@
 <contactref element="R3" pad="1"/>
 <wire x1="81.28" y1="56.515" x2="81.28" y2="54.24" width="1.27" layer="16"/>
-<wire x1="77.47" y1="60.96" x2="77.47" y2="63.5" width="0" layer="19" extent="1-1"/>
+<wire x1="77.47" y1="63.5" x2="77.47" y2="60.96" width="1.4224" layer="16"/>
+<contactref element="LED1" pad="A"/>
+<wire x1="77.47" y1="40.64" x2="78.74" y2="41.91" width="1.4224" layer="16"/>
+<wire x1="78.74" y1="41.91" x2="82.55" y2="41.91" width="1.4224" layer="16"/>
 </signal>
 </signals>
