File: psu/psu.sch (EAGLE design)
At the start: 39 parts, among them IC1 7815T, IC2 7915T, IC3 7812T, IC4 7912T, IC5 7805T, J1 15VAC, J2 POWER_SW

Commit message: Loading resistors for the PSU
Parts:
- added R1, R2, R3, R4, R5: 2.4k, SparkFun-Resistors:RESISTOR0805-RES
Connections:
- net +12V: now also R2.1
- net +15V: now also R1.1
- net +5V: now also R3.1
- net -12V: now also R4.1
- net -15V: now also R5.1
- net GND: now also R1.2, R2.2, R3.2, R4.2, R5.2
Other:
- note added: "(for all)"
- note added: "loading"

Commit message: psu rev 2: fix disconnected nets, add led
Parts:
- added LED1: (no value), led:LED3MM
Connections:
- net +5V: now also LED1.A
- net GND: now also LED1.C
Other:
- note added: "status"
Changed lines of the file:
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@@
 <?xml version="1.0" encoding="utf-8"?>
 <!DOCTYPE eagle SYSTEM "eagle.dtd">
-<eagle version="7.5.0">
+<eagle version="7.6.0">
 <drawing>
 <settings>
@@
 <grid distance="0.05" unitdist="inch" unit="inch" style="lines" multiple="1" display="no" altdistance="0.01" altunitdist="inch" altunit="inch"/>
 <layers>
-<layer number="1" name="Top" color="4" fill="1" visible="yes" active="no"/>
-<layer number="16" name="Bottom" color="1" fill="1" visible="yes" active="no"/>
-<layer number="17" name="Pads" color="2" fill="1" visible="yes" active="no"/>
-<layer number="18" name="Vias" color="2" fill="1" visible="yes" active="no"/>
-<layer number="19" name="Unrouted" color="6" fill="1" visible="yes" active="no"/>
-<layer number="20" name="Dimension" color="15" fill="1" visible="yes" active="no"/>
-<layer number="21" name="tPlace" color="16" fill="1" visible="yes" active="no"/>
-<layer number="22" name="bPlace" color="14" fill="1" visible="yes" active="no"/>
-<layer number="23" name="tOrigins" color="15" fill="1" visible="yes" active="no"/>
-<layer number="24" name="bOrigins" color="15" fill="1" visible="yes" active="no"/>
-<layer number="25" name="tNames" color="7" fill="1" visible="yes" active="no"/>
-<layer number="26" name="bNames" color="7" fill="1" visible="yes" active="no"/>
-<layer number="27" name="tValues" color="7" fill="1" visible="yes" active="no"/>
-<layer number="28" name="bValues" color="7" fill="1" visible="yes" active="no"/>
+<layer number="1" name="Top" color="4" fill="1" visible="no" active="no"/>
+<layer number="16" name="Bottom" color="1" fill="1" visible="no" active="no"/>
+<layer number="17" name="Pads" color="2" fill="1" visible="no" active="no"/>
+<layer number="18" name="Vias" color="2" fill="1" visible="no" active="no"/>
+<layer number="19" name="Unrouted" color="6" fill="1" visible="no" active="no"/>
+<layer number="20" name="Dimension" color="15" fill="1" visible="no" active="no"/>
+<layer number="21" name="tPlace" color="16" fill="1" visible="no" active="no"/>
+<layer number="22" name="bPlace" color="14" fill="1" visible="no" active="no"/>
+<layer number="23" name="tOrigins" color="15" fill="1" visible="no" active="no"/>
+<layer number="24" name="bOrigins" color="15" fill="1" visible="no" active="no"/>
+<layer number="25" name="tNames" color="7" fill="1" visible="no" active="no"/>
+<layer number="26" name="bNames" color="7" fill="1" visible="no" active="no"/>
+<layer number="27" name="tValues" color="7" fill="1" visible="no" active="no"/>
+<layer number="28" name="bValues" color="7" fill="1" visible="no" active="no"/>
 <layer number="29" name="tStop" color="7" fill="3" visible="no" active="no"/>
 <layer number="30" name="bStop" color="7" fill="6" visible="no" active="no"/>
@@
 <layer number="35" name="tGlue" color="7" fill="4" visible="no" active="no"/>
 <layer number="36" name="bGlue" color="7" fill="5" visible="no" active="no"/>
-<layer number="37" name="tTest" color="7" fill="1" visible="yes" active="no"/>
-<layer number="38" name="bTest" color="7" fill="1" visible="yes" active="no"/>
+<layer number="37" name="tTest" color="7" fill="1" visible="no" active="no"/>
+<layer number="38" name="bTest" color="7" fill="1" visible="no" active="no"/>
 <layer number="39" name="tKeepout" color="4" fill="11" visible="no" active="no"/>
 <layer number="40" name="bKeepout" color="1" fill="11" visible="no" active="no"/>
@@
 <layer number="44" name="Drills" color="7" fill="1" visible="no" active="no"/>
 <layer number="45" name="Holes" color="7" fill="1" visible="no" active="no"/>
-<layer number="46" name="Milling" color="3" fill="1" visible="yes" active="no"/>
-<layer number="47" name="Measures" color="7" fill="1" visible="yes" active="no"/>
-<layer number="48" name="Document" color="7" fill="1" visible="yes" active="no"/>
-<layer number="49" name="Reference" color="7" fill="1" visible="yes" active="no"/>
-<layer number="50" name="dxf" color="7" fill="1" visible="yes" active="no"/>
-<layer number="51" name="tDocu" color="6" fill="1" visible="yes" active="no"/>
-<layer number="52" name="bDocu" color="7" fill="1" visible="yes" active="no"/>
-<layer number="53" name="tGND_GNDA" color="7" fill="9" visible="yes" active="no"/>
-<layer number="54" name="bGND_GNDA" color="1" fill="9" visible="yes" active="no"/>
-<layer number="56" name="wert" color="7" fill="1" visible="yes" active="no"/>
-<layer number="57" name="tCAD" color="7" fill="1" visible="yes" active="no"/>
-<layer number="59" name="tCarbon" color="7" fill="1" visible="yes" active="no"/>
-<layer number="60" name="bCarbon" color="7" fill="1" visible="yes" active="no"/>
+<layer number="46" name="Milling" color="3" fill="1" visible="no" active="no"/>
+<layer number="47" name="Measures" color="7" fill="1" visible="no" active="no"/>
+<layer number="48" name="Document" color="7" fill="1" visible="no" active="no"/>
+<layer number="49" name="Reference" color="7" fill="1" visible="no" active="no"/>
+<layer number="50" name="dxf" color="7" fill="1" visible="no" active="no"/>
+<layer number="51" name="tDocu" color="6" fill="1" visible="no" active="no"/>
+<layer number="52" name="bDocu" color="7" fill="1" visible="no" active="no"/>
+<layer number="53" name="tGND_GNDA" color="7" fill="9" visible="no" active="no"/>
+<layer number="54" name="bGND_GNDA" color="1" fill="9" visible="no" active="no"/>
+<layer number="56" name="wert" color="7" fill="1" visible="no" active="no"/>
+<layer number="57" name="tCAD" color="7" fill="1" visible="no" active="no"/>
+<layer number="59" name="tCarbon" color="7" fill="1" visible="no" active="no"/>
+<layer number="60" name="bCarbon" color="7" fill="1" visible="no" active="no"/>
 <layer number="90" name="Modules" color="5" fill="1" visible="yes" active="yes"/>
 <layer number="91" name="Nets" color="2" fill="1" visible="yes" active="yes"/>
@@
 <part name="R4" library="SparkFun-Resistors" deviceset="RESISTOR" device="0805-RES" value="2.4k"/>
 <part name="R5" library="SparkFun-Resistors" deviceset="RESISTOR" device="0805-RES" value="2.4k"/>
+<part name="LED1" library="led" deviceset="LED" device="3MM"/>
+<part name="GND11" library="supply1" deviceset="GND" device=""/>
 </parts>
 <sheets>
@@
 <wire x1="191.77" y1="34.29" x2="200.66" y2="34.29" width="0.1524" layer="97"/>
 <wire x1="200.66" y1="34.29" x2="200.66" y2="38.1" width="0.1524" layer="97"/>
-<wire x1="245.11" y1="0" x2="245.11" y2="38.1" width="0.1524" layer="97"/>
+<wire x1="245.11" y1="0" x2="245.11" y2="21.59" width="0.1524" layer="97"/>
+<wire x1="245.11" y1="21.59" x2="245.11" y2="25.4" width="0.1524" layer="97"/>
+<wire x1="245.11" y1="25.4" x2="245.11" y2="38.1" width="0.1524" layer="97"/>
 <wire x1="245.11" y1="66.04" x2="255.27" y2="66.04" width="0.1524" layer="97"/>
 <wire x1="255.27" y1="66.04" x2="278.13" y2="66.04" width="0.1524" layer="97"/>
-<wire x1="278.13" y1="66.04" x2="278.13" y2="0" width="0.1524" layer="97"/>
+<wire x1="278.13" y1="66.04" x2="278.13" y2="25.4" width="0.1524" layer="97"/>
+<wire x1="278.13" y1="25.4" x2="278.13" y2="0" width="0.1524" layer="97"/>
 <wire x1="278.13" y1="0" x2="245.11" y2="0" width="0.1524" layer="97"/>
 <text x="246.38" y="63.5" size="1.778" layer="97">loading</text>
@@
 <wire x1="255.27" y1="62.23" x2="255.27" y2="66.04" width="0.1524" layer="97"/>
 <text x="268.478" y="58.9026" size="1.27" layer="96">(for all)</text>
+<wire x1="245.11" y1="25.4" x2="254" y2="25.4" width="0.1524" layer="97"/>
+<wire x1="254" y1="25.4" x2="278.13" y2="25.4" width="0.1524" layer="97"/>
+<wire x1="245.11" y1="21.59" x2="254" y2="21.59" width="0.1524" layer="97"/>
+<wire x1="254" y1="21.59" x2="254" y2="25.4" width="0.1524" layer="97"/>
+<text x="246.38" y="22.86" size="1.778" layer="97">status</text>
 </plain>
 <instances>
@@
 <attribute name="NAME" x="259.08" y="48.4886" size="1.778" layer="95"/>
 </instance>
+<instance part="LED1" gate="G$1" x="259.08" y="12.7" rot="R90"/>
+<instance part="GND11" gate="1" x="269.24" y="7.62"/>
 </instances>
 <busses>
@@
 <junction x="270.51" y="36.83"/>
 </segment>
+<segment>
+<pinref part="LED1" gate="G$1" pin="C"/>
+<pinref part="GND11" gate="1" pin="GND"/>
+<wire x1="264.16" y1="12.7" x2="269.24" y2="12.7" width="0.1524" layer="91"/>
+<wire x1="269.24" y1="12.7" x2="269.24" y2="10.16" width="0.1524" layer="91"/>
+</segment>
 </net>
 <net name="+AC" class="0">
@@
 <label x="256.54" y="41.91" size="1.27" layer="95" rot="R180" xref="yes"/>
 </segment>
+<segment>
+<pinref part="LED1" gate="G$1" pin="A"/>
+<wire x1="252.73" y1="12.7" x2="256.54" y2="12.7" width="0.1524" layer="91"/>
+<label x="252.73" y="12.7" size="1.27" layer="95" rot="R180" xref="yes"/>
+</segment>
 </net>
