File: vco-4069-schmitz/vco-4069-schmitz.brd (EAGLE design)
At the start: 58.4 x 36.8 mm, 46 parts, among them IC1 4069N, J1 22k pot (fp), J2 22k pot (fp), Q1 BC560, Q2 BC550B, Q3 BC550B

Commit message: bump and add board bom
Parts:
- moved R1 1.27 mm to (19.1, 29.2)
- moved R2 1.27 mm to (15.9, 29.2)
- moved R6 1.27 mm to (12.7, 29.2)
- moved R3 0.89 mm to (19.1, 24.9)
- moved R4 0.89 mm to (15.9, 24.9)
- moved R7 0.89 mm to (12.7, 24.9)
Routing:
- net N$1: track 10.5 -> 8.74 mm
- net N$8: track 40.3 -> 41.4 mm
Other:
- board text added: "4069vco 2016/iwx"
